File: V1/PCB/ElectronThingyStick.sch (EAGLE design)
At the start: 105 parts, among them T2 BC847

Commit message: Corrected electron name and minor tidyup.
Added pdfs of the PCB.

Added BOM to list the parts
Parts:
- removed U$1: ELECTRONDUALROW, Tinamous:ELECTRONDUALROW
- added IC1: ELECTRONDUALROW, Tinamous:ELECTRONDUALROW
Connections:
- net 3.3V: now also IC1.3V3; no longer U$1.3V3
- net 5V: now also IC1.VIN; no longer U$1.VIN
- net GND: now also IC1.GND, IC1.GND@2; no longer U$1.GND, U$1.GND@2
- net N$1: now also IC1.C5; no longer U$1.C5
- net N$10: now also IC1.A3; no longer U$1.A3
- net N$11: now also IC1.A2; no longer U$1.A2
- net N$12: now also IC1.A1; no longer U$1.A1
- net N$13: now also IC1.A0; no longer U$1.A0
- net N$15: now also IC1.C2; no longer U$1.C2
- net N$16: now also IC1.D5; no longer U$1.D5
- net N$17: now also IC1.D4; no longer U$1.D4
- net N$18: now also IC1.D3; no longer U$1.D3
- net N$19: now also IC1.D2; no longer U$1.D2
- net N$20: now also IC1.D1; no longer U$1.D1
- net N$21: now also IC1.D0; no longer U$1.D0
- net N$22: now also IC1.B5; no longer U$1.B5
- net N$24: now also IC1.!RST; no longer U$1.!RST
- net N$25: now also IC1.C1; no longer U$1.C1
- net N$27: now also IC1.C0; no longer U$1.C0
- net N$32: now also IC1.B4; no longer U$1.B4
- net N$35: now also IC1.B3; no longer U$1.B3
- net N$38: now also IC1.D7; no longer U$1.D7
- net N$39: now also IC1.D6; no longer U$1.D6
- net N$4: now also IC1.C4; no longer U$1.C4
- net N$41: now also IC1.B2; no longer U$1.B2
- net N$44: now also IC1.B1; no longer U$1.B1
- net N$45: now also IC1.B0; no longer U$1.B0
- net N$5: now also IC1.C3; no longer U$1.C3
- net N$6: now also IC1.WKP; no longer U$1.WKP
- net N$7: now also IC1.DAC; no longer U$1.DAC
- net N$8: now also IC1.A5; no longer U$1.A5
- net N$9: now also IC1.A4; no longer U$1.A4
- net RX: now also IC1.RX; no longer U$1.RX
- net TX: now also IC1.TX; no longer U$1.TX
- net V_BATT: now also IC1.VBAT; no longer U$1.VBAT
Other:
- moved on the sheet: C1, H2, H3, H4, JP1, JP10, JP11, JP13, JP14, JP15, JP16, JP17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
